File: MPF2VGA.kicad_sch (KiCad schematic)
At the start: 33 parts, among them IC1 EPM7128SLC84-15, J1 DSUB_HD15, J2 JTAG, U1 MS62256A-35NC, X1 25.175

Commit message: Fix capacitors
Parts:
- BUS2: value MPF2 II BUS -> MPF II BUS
- C11, C2, C3, C4, C5, C6, C7, C8, C9: value 0.01 -> 0.1u
Changed lines of the file:
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@@
       (effects (font (size 1.524 1.524)))
     )
-    (property "Value" "MPF2 II BUS" (at 54.61 59.9581 0)
+    (property "Value" "MPF II BUS" (at 54.61 59.9581 0)
       (effects (font (size 1.524 1.524)))
     )
@@
       (effects (font (size 1.27 1.27)) (justify left))
     )
-    (property "Value" "0.01" (at 103.251 215.9073 0)
+    (property "Value" "0.1u" (at 103.251 215.9073 0)
       (effects (font (size 1.27 1.27)) (justify left))
     )
@@
       (effects (font (size 1.27 1.27)) (justify left))
     )
-    (property "Value" "0.01" (at 58.801 215.9073 0)
+    (property "Value" "0.1u" (at 58.801 215.9073 0)
       (effects (font (size 1.27 1.27)) (justify left))
     )
@@
       (effects (font (size 1.27 1.27)) (justify left))
     )
-    (property "Value" "0.01" (at 67.691 215.9073 0)
+    (property "Value" "0.1u" (at 67.691 215.9073 0)
       (effects (font (size 1.27 1.27)) (justify left))
     )
@@
       (effects (font (size 1.27 1.27)) (justify left))
     )
-    (property "Value" "0.01" (at 85.471 215.9073 0)
+    (property "Value" "0.1u" (at 85.471 215.9073 0)
       (effects (font (size 1.27 1.27)) (justify left))
     )
@@
       (effects (font (size 1.27 1.27)) (justify left))
     )
-    (property "Value" "0.01" (at 48.641 215.9073 0)
+    (property "Value" "0.1u" (at 48.641 215.9073 0)
       (effects (font (size 1.27 1.27)) (justify left))
     )
@@
       (effects (font (size 1.27 1.27)) (justify left))
     )
-    (property "Value" "0.01" (at 121.031 215.9073 0)
+    (property "Value" "0.1u" (at 121.031 215.9073 0)
       (effects (font (size 1.27 1.27)) (justify left))
     )
@@
       (effects (font (size 1.27 1.27)) (justify left))
     )
-    (property "Value" "0.01" (at 112.141 215.9073 0)
+    (property "Value" "0.1u" (at 112.141 215.9073 0)
       (effects (font (size 1.27 1.27)) (justify left))
     )
@@
       (effects (font (size 1.27 1.27)) (justify left))
     )
-    (property "Value" "0.01" (at 94.361 215.9073 0)
+    (property "Value" "0.1u" (at 94.361 215.9073 0)
       (effects (font (size 1.27 1.27)) (justify left))
     )
@@
       (effects (font (size 1.27 1.27)) (justify left))
     )
-    (property "Value" "0.01" (at 76.581 215.9073 0)
-      (effects (font (size 1.27 1.27)) (justify left))
-    )
+    (property "Value" "0.1u" (at 76.581 215.9073 0)
+      (effects (font (size 1.27 1.27)) (justify left))
+    )
